File: 006P-5V-3V3Supply.brd (EAGLE design)
At the start: 69.5 x 34.3 mm, 15 parts, among them IC1 7805T, IC2 TM48M033F

Commit message: 回路図、基板図を修正
Parts:
- D1, D2: value 1N4004 -> 1N4007
- R1: value 1k -> 10k
Changed lines of the file:
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@@
 <element name="C6" library="rcl" package="C025-024X044" value="0.1uF" x="41.91" y="20.32" rot="R180"/>
 <element name="C7" library="rcl" package="C025-024X044" value="0.1uF" x="46.99" y="20.32" rot="R180"/>
-<element name="D1" library="diode" package="DO41-10" value="1N4004" x="27.94" y="5.08"/>
-<element name="D2" library="diode" package="DO41-10" value="1N4004" x="45.72" y="15.24"/>
+<element name="D1" library="diode" package="DO41-10" value="1N4007" x="27.94" y="5.08"/>
+<element name="D2" library="diode" package="DO41-10" value="1N4007" x="45.72" y="15.24"/>
 <element name="IC1" library="linear" package="TO220H" value="7805T" x="27.94" y="22.86"/>
 <element name="IC2" library="linear" package="TO220V" value="TM48M033F" x="45.72" y="20.32"/>
@@
 <attribute name="OC_FARNELL" value="unknown" x="55.88" y="17.78" size="1.778" layer="28" rot="MR270" display="off"/>
 </element>
-<element name="R1" library="rcl" package="0207/7" value="1k" x="16.51" y="17.78"/>
+<element name="R1" library="rcl" package="0207/7" value="10k" x="16.51" y="17.78"/>
 <element name="LED1" library="led" package="LED3MM" value="" x="12.7" y="13.97" rot="R270"/>
 <element name="9VIN" library="con-wago-508" package="W237-132" value="" x="5.08" y="17.78" rot="R270">
